File: mixer.kicad_sch (KiCad schematic)
At the start: 52 parts, among them U1 TLV3501AID, U2 TLV9062, U3 TLV3501AID, U4 TLV9062, U5 TLV9062, U6 OPA2192, U7 ADG779

Commit message: added r/c values
Parts:
- added C22, C23, C24: 100n, symbol Device:C
- C1, C2: value C -> 2.2n
- C10, C11, C12, C13, C14, C18, C19, C20, C21, C3, C4, C5, C6, C9: value C -> 100n
- C15: value C -> 47n
- C16: value C -> 22n
- C17, C7, C8: value C -> 10n
- R1, R11, R12, R14, R15, R19, R2, R20, R3: value R -> 10k
- R10: value R -> 6k
- R13, R9: value R -> 4.7k
- R16: value R -> 3k
- R17: value R -> 1.5k
- R18: value R -> 6.8k
- R21, R22: value R -> 100k
- R4: value R -> 8.2k
- R5: value R -> 200k
- R6: value R -> 500k
- R7, R8: value R -> 1M
- RV1: value R_Potentiometer -> 20k
- RV2: value R_Potentiometer -> 1k
Connections:
- net +2V5: now also U3.7 (V+), C22.2
- net -2V5: now also U3.4 (V-), U3.8 (SHDN), C23.1
- net GND: now also C22.1, C23.2, C24.1
- net at R21.2, RV1.2: now also C24.2
Other:
- moved on the sheet: RV1
